File: pcb/hhkb_split_left.kicad_sch (KiCad schematic)
At the start: 66 parts, among them SW1 keyswitch, SW10 keyswitch, SW11 keyswitch, SW12 keyswitch, SW13 keyswitch, SW14 keyswitch, SW15 keyswitch, SW16 keyswitch, SW17 keyswitch, SW18 keyswitch, SW19 keyswitch, SW2 keyswitch, SW20 keyswitch, SW21 keyswitch, SW22 keyswitch, SW23 keyswitch, SW24 keyswitch, SW25 keyswitch, SW26 keyswitch, SW27 keyswitch, SW3 keyswitch, SW4 keyswitch, SW5 keyswitch, SW6 keyswitch, SW7 keyswitch, SW8 keyswitch, SW9 keyswitch, U1 74LVC595

Commit message: 回路図のバス配線を「部品ごとに枝を引く」方式に固め、可読性の指摘に応えた（指摘1）
同じネット（V3V3・GND）を1本のバスから各部品へ枝で配る方式に、
以下の防御を加えて安定させた。

- 枝は「先に横、それから縦」で描き、ピンの列を素通りしない
  （同じ部品が V3V3・GND を両方持つ場合、隣接ピンを串刺しにして
  無関係なネットに誤統合される事故が3回起きた）
- バスの枝は全部品を置き終えたあとに一括で描く
  （グループの処理順に依存する短絡を避ける）
- ピンピッチを 2.54mm→5.08mm に広げ、グローバルラベルの矢印が
  隣どうしで重ならないようにした（1.27mmグリッドの整数倍を維持）

利用者のスクリーンショット指摘（上下バスが同じ足につながって見える・
V3V3ラベルとCOL0ラベルの文字が重なる）を実測で確認し、解消した。

確認: test_schematic.py 9件全通過。ERC の multiple_net_names・
pin_to_pin エラーは複数回の再生成で0件。netlist の最大ノードは
GND=12（以前は69ノードの巨大ネット化バグがあった）。
Connections:
- net GND is gone; now on net V3V3: BT1_-.1, C_BULK.2, C_RAIL.2, C_U1.2, J_DB.12, J_DB.2, R_LO.2, U1.13 (OE), U1.8 (GND)
- net VBATT_SW is gone; now on net VBATT_SENSE: D_PWR.2 (A), R_HI.1, SW_PWR_2.1
Other:
- moved on the sheet: BT1_+, BT1_-, C_BULK, C_RAIL, C_U1, D1, D10, D11, D12, D13, D14, D15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
