File: pcb/hhkb_split_right.kicad_sch (KiCad schematic)
At the start: 82 parts, among them SW1 keyswitch, SW10 keyswitch, SW11 keyswitch, SW12 keyswitch, SW13 keyswitch, SW14 keyswitch, SW15 keyswitch, SW16 keyswitch, SW17 keyswitch, SW18 keyswitch, SW19 keyswitch, SW2 keyswitch, SW20 keyswitch, SW21 keyswitch, SW22 keyswitch, SW23 keyswitch, SW24 keyswitch, SW25 keyswitch, SW26 keyswitch, SW27 keyswitch, SW28 keyswitch, SW29 keyswitch, SW3 keyswitch, SW30 keyswitch, SW31 keyswitch, SW32 keyswitch, SW33 keyswitch, SW34 keyswitch, SW4 keyswitch, SW5 keyswitch, SW6 keyswitch, SW7 keyswitch, SW8 keyswitch, SW9 keyswitch, U1 74LVC595, U2 74LVC595

Commit message: 回路図のバス配線を「部品ごとに枝を引く」方式に固め、可読性の指摘に応えた（指摘1）
同じネット（V3V3・GND）を1本のバスから各部品へ枝で配る方式に、
以下の防御を加えて安定させた。

- 枝は「先に横、それから縦」で描き、ピンの列を素通りしない
  （同じ部品が V3V3・GND を両方持つ場合、隣接ピンを串刺しにして
  無関係なネットに誤統合される事故が3回起きた）
- バスの枝は全部品を置き終えたあとに一括で描く
  （グループの処理順に依存する短絡を避ける）
- ピンピッチを 2.54mm→5.08mm に広げ、グローバルラベルの矢印が
  隣どうしで重ならないようにした（1.27mmグリッドの整数倍を維持）

利用者のスクリーンショット指摘（上下バスが同じ足につながって見える・
V3V3ラベルとCOL0ラベルの文字が重なる）を実測で確認し、解消した。

確認: test_schematic.py 9件全通過。ERC の multiple_net_names・
pin_to_pin エラーは複数回の再生成で0件。netlist の最大ノードは
GND=12（以前は69ノードの巨大ネット化バグがあった）。
Connections:
- net COL2 is gone; now on net COL1: SW19.1, SW26.1, SW3.1, SW32.1, U1.2 (Q2)
- net COL3 is gone; now on net COL1: SW12.1, SW20.1, SW27.1, SW4.1, U1.3 (Q3)
- net COL4 is gone; now on net COL1: SW13.1, SW21.1, SW28.1, SW33.1, SW5.1, U1.4 (Q4)
- net COL5 is gone; now on net COL1: SW14.1, SW22.1, SW29.1, SW34.1, SW6.1, U1.5 (Q5)
- net COL6 is gone; now on net COL1: SW15.1, SW23.1, SW7.1, U1.6 (Q6)
- net COL7 is gone; now on net COL1: SW16.1, SW24.1, SW30.1, SW8.1, U1.7 (Q7)
- net GND is gone; now on net V3V3: BT1_-.1, C_BULK.2, C_RAIL.2, C_U1.2, C_U2.2, J_DB.12, J_DB.2, R_LO.2, U1.13 (OE), U1.8 (GND), U2.13 (OE), U2.8 (GND)
- net U1_U2 is gone; now on net COL1: U1.9 (Q7S), U2.14 (DS)
- net VBATT_SW is gone; now on net VBATT_SENSE: D_PWR.2 (A), R_HI.1, SW_PWR_2.1
Other:
- moved on the sheet: BT1_+, BT1_-, C_BULK, C_RAIL, C_U1, C_U2, D1, D10, D11, D12, D13, D14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
