File: pcb/hhkb_split_right.kicad_sch (KiCad schematic)
At the start: 80 parts, among them SW1 keyswitch, SW10 keyswitch, SW11 keyswitch, SW12 keyswitch, SW13 keyswitch, SW14 keyswitch, SW15 keyswitch, SW16 keyswitch, SW17 keyswitch, SW18 keyswitch, SW19 keyswitch, SW2 keyswitch, SW20 keyswitch, SW21 keyswitch, SW22 keyswitch, SW23 keyswitch, SW24 keyswitch, SW25 keyswitch, SW26 keyswitch, SW27 keyswitch, SW28 keyswitch, SW29 keyswitch, SW3 keyswitch, SW30 keyswitch, SW31 keyswitch, SW32 keyswitch, SW33 keyswitch, SW34 keyswitch, SW4 keyswitch, SW5 keyswitch, SW6 keyswitch, SW7 keyswitch, SW8 keyswitch, SW9 keyswitch, U1 74LVC595, U2 74LVC595

Commit message: VBATT_RAW を廃止し、V3V3 を FFC の隙間を通る幅に直した
1. 電池の + を基板に通さない（利用者の指摘）
   BT1.+ →(VBATT_RAW)→ SW_PWR.1 と基板を往復させていたが、電池
   ボックスもスイッチもリード線で繋ぐので、+ はスイッチへ直接
   はんだ付けすればよい。線 4→3 本・ランド 4→2 個。基板から
   VBATT_RAW というネットが丸ごと消えた。
   ランドの数は WIRE_PAD_KINDS で 2 に決め打ちしていたのを、
   宣言した端子の数から取るように直した。参照名の接尾辞は端子数に
   関わらず付ける（1 個になった瞬間に BT1 へ化けて board_refs と
   回路図の配置表が一斉にずれるため）。

2. V3V3 の線幅 0.3 → 0.2mm ★右の V3V3 断線の真因
   「FFC の 0.30mm パッドに届く必要がある」と書いてあったが、
   **パッドの幅とパッドの隙間を取り違えていた。**0.5mm ピッチ・
   パッド幅 0.30 の列を幅 0.30 で抜けると隣のパッドまで 0.200mm
   ちょうどで、丸めで即割る（0.20mm なら 0.250mm で通る）。
   右基板で V3V3 だけが J_DB から出られず、自動配線器がビアだけ
   (72.75, 84.00) に置いて両端とも繋がず放棄していた。同じ列の
   VBATT_SENSE・SPI_MOSI・SCK・CS は全部 0.20mm で脱出できていた。
   電流は BLE のパルスで 15mA、バルクは子基板側なのでこの線が
   運ぶのは平均電流だけ。0.20mm でも桁が違うほど余る。

3. DSN のクリアランスマージン 15 → 20µm
   上の変更のあと 15 では丸め不足が顕在化し、違反が左 1・右 3 出た
   （実測 0.1917〜0.1919mm ＜ 0.2000mm）。20 で全部消える。
   15/20/25 の結果は autoroute.py に表で残した。

結果:
  左  違反 0 / 未配線 2
  右  違反 0 / 未配線 0   ← 今日はじめて 0/0
  子  違反 0 / 未配線 0

左の 2 本は ROW3/ROW4 が J_DB へ降りる枝。**瑣末と判断**（利用者）。
J_DB の ROW パッドの並び（ROW3,ROW2,ROW1,ROW0,ROW4）が行バスの
y 順と食い違っていて交差する。XIAO のピン割り当てを変えて順序を
揃えれば解ける見込み——次の課題。

pytest tools は未実行。

Co-Authored-By: Claude Opus 5 (1M context) <noreply@anthropic.com>
Parts:
- removed BT1_+: battery_land, symbol hhkb_split_right:battery_land
- removed SW_PWR_2: wire_land, symbol hhkb_split_right:wire_land
Connections:
- net VBATT_RAW is gone; now on net VBATT_SENSE: SW_PWR_1.1
Other:
- moved on the sheet: BT1_-, C_U1, C_U2, D1, D10, D11, D12, D13, D14, D15, D16, D17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

Commit message: 電源を子基板へ移し、FFC のピン順を両基板の都合から決め直した
利用者が絵を見ながら出した指摘を順に潰した回。**私は数字だけ見て
絵を見ておらず、同じ型の見落としを何度も拾ってもらった。**

■ 電源部を子基板へ（open-gaps #41）

  消費者は XIAO で、それは子基板にいる。起動と BLE 初期化で
  2.0〜2.5mA を継続、送信で 10〜15mA のパルス（task-c4-c5 測定 C /
  electrical-design 1-5）。595 の走査 100µA とは 100 倍以上ちがう。
  主基板で整流すると、その mA 級が FFC の 0.2mm 1 本を 100mm 渡る。

    FFC の V3V3   2.0〜2.5mA 継続 + パルス → **約 100µA**（150 分の 1）
    VBATT_SENSE   500kΩ が 100mm 渡る     → **渡らない**（ADC の 2mm 隣）
    ショットキー  隔離点まで FFC 100mm     → **3V3 パッド直近**
    主基板の帯    電源 5 点が SPI を塞ぐ   → **空いた**

  電池もスイッチも子基板のすぐ隣（実測: スイッチ→縁 左 4.0 / 右 20.7mm）
  なのでリード線はむしろ短くなる。

■ FFC のピン順（利用者「DB 単体でなく MAIN の都合も視野に入れて」）

  ROW0/1 は J_DB より上、ROW2/3/4 は下へ伸びる。行番号の昇順に並べると
  上下 2 群が必ず交差する（**実測 3 交差**）。群ごとに近い順で **0 交差**。
  そのズレは **XIAO のピン割り当て＝ファームで吸収**する（利用者の判断
  「配線でひねるのではなくソフトで受けるべき」）。

  ROW4 を D9 から左列へ戻した。右列へ逃がしていた理由は「左列が 6 本だと
  アンテナ直下を 2 本通る」だが、**その 6 本目は VBATT_SENSE だった。**
  分圧が子基板へ移って 5 本に戻ったので前提が消えた。
  → ファームの `&spi2_default`（MISO 外し）が**不要になり削除**。

■ アンテナの禁止域（利用者「こんなに広い必要ある？」「ズレてる」）

  子基板: 幅 18.3mm（XIAO の外形）を使っていた。**アンテナは 3.5mm 角**で
  4.1 倍。さらに y 方向に 2 つの細工（意味の無い切り詰めと水増し）があり、
  **アンテナの 57% しか覆っていなかった**。
    → `antenna_x_band()` に統一。**被覆 100%**、地板の無駄も消えた。
  主基板: アンテナから 3.9mm 外れた場所を抜いて 450mm² を捨てていた。
    → 削除（前のコミット）。

  ⚠️ **SES 往復でルール領域の層が消える**ことを発見した（GetLayer() が -1）。
  層を持たないゾーンは何も禁止しないので、あとから敷いたベタが
  アンテナ直下に入っていた（実測 3297 頂点）。`_restore_rule_area_layers`
  で戻す。**「宣言したから効いている」の 3 回目。**

■ 子基板を主基板と同じ水準に（利用者「MAIN にあって DB に無いもの」）

  両面 GND ベタ（裏面だけだった）・GND ファンアウト・スティッチング・
  離島の救済・電源のネットクラス。順序は **配置 → ネットクラス → 配線 →
  ベタ・ビア**（利用者「ベタは配線の残りで最大限やる」）。
  アンテナの禁止域だけは最初（配置と配線の制約なので）。

■ その他

  - バルクを縦置き＋向きを直した（V3V3/GND が XIAO と平行に並ぶ）
  - 行を D2〜D6 にして D1 を空け、奥側に 2.54mm 作った

■ 検査（どれも故意に壊して落ちることを確認）

  - `test_the_row_order_matches_between_firmware_and_circuit`
    行 N がファームと回路で同じピンを指すか。**既存の検査は集合しか
    見ておらず、D4 と D6 を入れ替えても通っていた**
  - 禁止域の寸法をアンテナの実寸と照合
  - `test_there_is_a_bulk_capacitor` を「XIAO と同じ基板にあるか」に
  - 変異検査が子基板も壊せるように（バルク移設で空振りしていた）
  - 正規表現がゾーンを跨いで**ベタ自身を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
Parts:
- removed BT1_-: battery_land, symbol hhkb_split_right:battery_land
- removed D_PWR: schottky, symbol hhkb_split_right:schottky
- removed R_HI, R_LO: res_1M, symbol hhkb_split_right:res_1M
- removed SW_PWR_1: wire_land, symbol hhkb_split_right:wire_land
Connections:
- net VBATT_SENSE is gone; now on net ROW0: J_DB.7
- net ROW0: no longer J_DB.8
- net ROW1: now also J_DB.8; no longer J_DB.9
- net ROW2: now also J_DB.11; no longer J_DB.10
- net ROW3: now also J_DB.10; no longer J_DB.11
- net ROW4: now also J_DB.9; no longer J_DB.4
- net SPI_MOSI: now also J_DB.4; no longer J_DB.5
- net V3V3 renamed GND
- net GND: now also J_DB.5; no longer J_DB.6
- no-connect marks 8 -> 9
Other:
- note removed: "── 電源 ──"
- moved on the sheet: C_U1, C_U2, D1, D10, D11, D12, D13, D14, D15, D16, D17, D18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

Commit message: #49 オシロ用テストパッドを実装した（左 5・右 6・実装なしのランド）
利用者の決定（Yes）。信号は SPI_SCK / SPI_MOSI / CS / V3V3 / GND、右は
595 の数珠つなぎ U1_U2 も。ROW/COL はダイオードとソケットのパッドで
見られるので出さない。kind `testpoint` を回路宣言・pinmap・
parts.NOT_ASSEMBLED（BOM/CPL に出さない）・回路図の群・gen_pcb の
絶対座標配置（TP_PLACE・本番の板の空きを実測して決めた）に通した。

検査側の修正: TestPoint 系フットプリントの円コートヤードを
_courtyard_bbox が読めず「コートヤード無し」と誤判定していた（四角を
足したら自己交差になって発覚）→ fp_circle も読む。

残り: 各パッドから既存ネットへのスタブ（GND 以外）を利用者が引く
（左 4・右 5）。引くまで DRC の未配線がその本数ぶん残る。

Co-Authored-By: Claude Fable 5 <noreply@anthropic.com>
Parts:
- added TP1, TP2, TP3, TP4, TP5, TP6: testpoint, symbol hhkb_split_right:testpoint
Connections:
- net COL0: now also SW18.1, SW25.1, SW32.1
- net COL1: now also SW17.1, SW31.1, TP4.1; no longer SW18.1, SW25.1, SW32.1
- net COL8: no longer SW17.1, SW31.1
- net CS: now also J_DB.4, TP3.1; no longer J_DB.1
- net GND: now also J_DB.1, TP5.1, TP6.1; no longer J_DB.12, J_DB.5
- net SPI_MOSI: now also J_DB.3, TP2.1; no longer J_DB.4
- net SPI_SCK: now also J_DB.5, TP1.1; no longer J_DB.3
- net SPARE2: now reaches J_DB.6
- net ROW0 renamed ROW_C
- net ROW_C: now also J_DB.10; no longer J_DB.7
- net ROW1 renamed ROW_A
- net ROW2 renamed ROW_B
- net ROW_B: now also J_DB.9; no longer J_DB.11
- net ROW3 renamed ROW_D
- net ROW_D: now also J_DB.11; no longer J_DB.10
- net ROW4 renamed ROW_E
- net ROW_E: now also J_DB.12; no longer J_DB.9
- new net SPARE: J_DB.7
- no-connect marks 9 -> 8
Other:
- note added: "── テストパッド ──"
- moved on the sheet: D1, D10, D11, D12, D13, D14, D15, D16, D17, D18, D19, D2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

Commit message: Revert "#49 オシロ用テストパッドを実装した"——利用者が取り消しを決定
パッドから既存ネットへのスタブが引けず（利用者「試行錯誤したが諦める」）。
代案（利用者提案）: 既存のビアのレジストを剥がしてリード線を半田付けできる
ようにする。部品追加も配線も不要。別コミットで実装する。
検査側の修正（_courtyard_bbox が fp_circle も読む）だけは有用なので残す。

This reverts commits b8ea548 and 4f7bba2 (except the test improvement).

Co-Authored-By: Claude Fable 5 <noreply@anthropic.com>
Parts:
- removed TP1, TP2, TP3, TP4, TP5, TP6: testpoint, symbol hhkb_split_right:testpoint
Connections:
- net SPARE is gone; now on net ROW0: J_DB.7
- net COL0: no longer SW18.1, SW25.1, SW32.1
- net COL1: now also SW18.1, SW25.1, SW32.1; no longer SW17.1, SW31.1
- net COL8: now also SW17.1, SW31.1
- net CS: now also J_DB.1; no longer J_DB.4
- net GND: now also J_DB.12, J_DB.5; no longer J_DB.1
- net SPI_MOSI: now also J_DB.4; no longer J_DB.3
- net SPI_SCK: now also J_DB.3; no longer J_DB.5
- net ROW_A renamed ROW1
- net ROW_B renamed ROW2
- net ROW2: now also J_DB.11; no longer J_DB.9
- net ROW_C renamed ROW0
- net ROW0: no longer J_DB.10
- net ROW_D renamed ROW3
- net ROW3: now also J_DB.10; no longer J_DB.11
- net ROW_E renamed ROW4
- net ROW4: now also J_DB.9; no longer J_DB.12
- net SPARE2: no longer names the net of J_DB.6
- no-connect marks 8 -> 9
Other:
- note removed: "── テストパッド ──"
- moved on the sheet: D1, D10, D11, D12, D13, D14, D15, D16, D17, D18, D19, D2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
