File: pcb/hhkb_split_daughterboard.kicad_pcb (KiCad board)
At the start: 2 copper layers, 21 x 32 mm, 11 parts

Commit message: BOM の Value に内部識別名 (kind) をそのまま書いていたのを直した
fp.SetValue(kind) が FP_MAP のキー（cap_100u/schottky/ffc_12p/res_1M 等）
をそのまま基板の Value に書いていた。kind はフットプリントを引くための
内部名で、部品の型番でも規格値でもない。JLCPCB の部品マッチはこの
Value 欄を見るので、schottky/ffc_12p/res_1M が「該当部品なし」の
赤字（要手動選定）になっていた（cap_100u/cap_100n は数字が近い分
コメント不一致の警告で済んでいた）。

ELEC_FP の各エントリに 3 要素目として実際の Value 文字列を追加し、
gen_pcb.py・gen_daughterboard.py の SetValue(kind) を SetValue(value) に
変更。値は parts-audit.md に確定記録済みの型番・規格をそのまま使った
（B5819W・FH12-12S-0.5SH(55)・1M・100nF・100uF）。

配線済みの pcb/*.kicad_pcb は Value フィールドのみをテキスト置換で
書き換え、座標・配線・UUID は一切触っていない（gen_pcb.py の再実行は
Freerouting 前の配置が変わり配線をやり直す必要が出るため避けた）。
left・daughterboard は DRC 0 を確認。right は未配線 1 件が残るが、
これは今回の変更前から一貫して存在する既存の問題（open-gaps.md に
別途記録）。

pcb/unrouted/ は gen_pcb.py の再実行で座標・UUID が全面的に再採番され
巨大な差分になるため、今回はコミットに含めていない。
Parts:
- D_PWR: value schottky -> B5819W
- R_HI, R_LO: value res_1M -> 1M
Changed lines of the file:
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@@
 			)
 		)
-		(property "Value" "res_1M"
+		(property "Value" "1M"
 			(at 0 -1.65 0)
 			(layer "B.Fab")
@@
 			)
 		)
-		(property "Value" "schottky"
+		(property "Value" "B5819W"
 			(at 0 -2.1 0)
 			(layer "B.Fab")
@@
 			)
 		)
-		(property "Value" "res_1M"
+		(property "Value" "1M"
 			(at 0 -1.65 90)
 			(layer "B.Fab")
