File: pcb/hhkb_split_daughterboard.kicad_sch (KiCad schematic)
At the start: 3 parts

Commit message: バルクを子基板へ移し、電源鎖を消費側へ寄せ、行バスを直線にした
利用者の指摘を順に潰した。どれも「測ったら前提が違っていた」型。

1. バルク（C_BULK）を子基板へ
   守る相手は XIAO の µs 級の電流変動（electrical-design 1-5）で、
   595 でも整流点でもない。XIAO は子基板にいるので、主基板に置くと
   FFC 100mm のインダクタンスの外側から供給することになる。
   XIAO の 3V3 パッドから 2.04mm の位置へ移した。

2. 電源ブロックを V3V3 の消費側へ
   整流点 D_PWR が板の左端にあるのに、消費側（C_U1・U1・J_DB）は
   全部反対側だった。U1 の左へ寄せて V3V3 の銅 132→81mm、
   VBATT_SENSE 110→78mm。左の帯 0 はアンテナ禁止域と取付穴で
   分断されていて、プラス側へは出せない（一度出して DRC 13 件）。

3. 行のバスを裏面の直線で自分で引く（prewire_row_bus）
   ROW0 が 222mm・ビア 7 本・区間 54 で表裏を行き来していた。
   同じ行のダイオードの K 側は y が完全に一致し、ライン上に
   スルーホールが無いので直線が引ける（ROW4 は元から 0 ビアだった）。
   左の未配線 1 本（ROW2）はこれで解決した。
   ⚠️ DSN に (autoroute_settings) を足す道は駄目。左が 66 本に壊れた。

4. アンテナの禁止域（30x15mm）を削除
   利用者の「本当にアンテナの真上ですか」で測ったら、覆っていなかった。
     禁止域 y 30.60..45.60 / 基板後端 48.70 / アンテナ 49.50..53.00
   アンテナは基板の後端より 0.80mm 奥（XIAO_OVERHANG 1.8mm の効果）で、
   平面的に基板の外。禁止域は 3.9mm 的を外したまま 450mm² を捨て、
   左の配線を圧迫していた。
   **根拠に挙げられていた検査は存在しなかった。**interface.py は
   test_the_antenna_keepout_actually_covers_the_antenna が照合すると
   書いていたが、その名前の検査はどこにも無い。実在したのは
   「禁止域の中が空か」だけで、位置は誰も見ていなかった。
   代わりに test_the_antenna_clears_the_main_board を置いた
   （XIAO_OVERHANG を 0 にすると落ちることを確認済み）。

   → open-gaps #23 の幾何の証明（アンテナは必ず 4mm 以上 基板の下に
     入る）は、もう成立していない。ただし余裕は 0.80mm しかないので、
     手 0（アルミ箔で RSSI）の価値は残る。#23 の書き直しは次。

残っているもの（次に着手する）:
  右 未配線 3（GND 離島 1 + V3V3 が J_DB へ届かない 2）★機能的な故障
  左 未配線 1（GND 離島）
  違反はどれも 0。自前配線で塞ぐ案は取らない——今は綺麗に引けても
  配置を変えると黙って壊れ、再現性が無い（利用者の判断）。

pytest tools は未実行。

Co-Authored-By: Claude Opus 5 (1M context) <noreply@anthropic.com>
Parts:
- added C_BULK: cap_100u, symbol hhkb_split_daughterboard:cap_100u
Connections:
- net GND: now also C_BULK.2
- net V3V3: now also C_BULK.1
Changed lines of the file:
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@@
 	(generator "hhkb_split")
 	(generator_version "10.0")
-	(paper "User" 234.95 411.48)
+	(paper "User" 295.91 411.48)
 	(title_block
 		(title "hhkb_split_daughterboard")
@@
 	)
 	(wire
-		(pts (xy 58.42 43.18) (xy 124.46 43.18))
+		(pts (xy 58.42 43.18) (xy 185.42 43.18))
 		(stroke (width 0.508) (type default))
 	)
@@
 	)
 	(wire
-		(pts (xy 58.42 175.26) (xy 124.46 175.26))
+		(pts (xy 58.42 175.26) (xy 185.42 175.26))
 		(stroke (width 0.508) (type default))
 	)
@@
 	)
 	(wire
+		(pts (xy 185.42 96.52) (xy 180.34 96.52))
+		(stroke (width 0) (type default))
+	)
+	(wire
+		(pts (xy 180.34 96.52) (xy 180.34 43.18))
+		(stroke (width 0) (type default))
+	)
+	(wire
+		(pts (xy 180.34 43.18) (xy 185.42 43.18))
+		(stroke (width 0) (type default))
+	)
+	(junction (at 185.42 43.18) (diameter 1.016) (color 0 0 0 0)
+	)
+	(wire
 		(pts (xy 63.50 160.02) (xy 58.42 160.02))
 		(stroke (width 0) (type default))
@@
 	)
 	(junction (at 124.46 175.26) (diameter 1.016) (color 0 0 0 0)
+	)
+	(wire
+		(pts (xy 185.42 101.60) (xy 180.34 101.60))
+		(stroke (width 0) (type default))
+	)
+	(wire
+		(pts (xy 180.34 101.60) (xy 180.34 175.26))
+		(stroke (width 0) (type default))
+	)
+	(wire
+		(pts (xy 180.34 175.26) (xy 185.42 175.26))
+		(stroke (width 0) (type default))
+	)
+	(junction (at 185.42 175.26) (diameter 1.016) (color 0 0 0 0)
 	)
 	(wire
@@
 					(unit 1)
 				)
+			)
+		)
+	)
+	(symbol
+		(lib_id "hhkb_split_daughterboard:cap_100u")
+		(at 196.85 99.06 0)
+		(unit 1)
+		(exclude_from_sim no)
+		(in_bom yes)
+		(on_board yes)
+		(dnp no)
+		(property "Reference" "C_BULK" (at 196.85 87.63 0) (effects (font (size 1.27 1.27))))
+		(property "Value" "cap_100u" (at 196.85 110.49 0) (effects (font (size 1.27 1.27))))
+		(pin "1")
+		(pin "2")
+		(instances
+			(project "hhkb_split_daughterboard"
+				(path "/569e6ce2-5cbf-5b99-8a67-ce450b40985c"
+					(reference "C_BULK")
+					(unit 1)
+				)

Commit message: 電源を子基板へ移し、FFC のピン順を両基板の都合から決め直した
利用者が絵を見ながら出した指摘を順に潰した回。**私は数字だけ見て
絵を見ておらず、同じ型の見落としを何度も拾ってもらった。**

■ 電源部を子基板へ（open-gaps #41）

  消費者は XIAO で、それは子基板にいる。起動と BLE 初期化で
  2.0〜2.5mA を継続、送信で 10〜15mA のパルス（task-c4-c5 測定 C /
  electrical-design 1-5）。595 の走査 100µA とは 100 倍以上ちがう。
  主基板で整流すると、その mA 級が FFC の 0.2mm 1 本を 100mm 渡る。

    FFC の V3V3   2.0〜2.5mA 継続 + パルス → **約 100µA**（150 分の 1）
    VBATT_SENSE   500kΩ が 100mm 渡る     → **渡らない**（ADC の 2mm 隣）
    ショットキー  隔離点まで FFC 100mm     → **3V3 パッド直近**
    主基板の帯    電源 5 点が SPI を塞ぐ   → **空いた**

  電池もスイッチも子基板のすぐ隣（実測: スイッチ→縁 左 4.0 / 右 20.7mm）
  なのでリード線はむしろ短くなる。

■ FFC のピン順（利用者「DB 単体でなく MAIN の都合も視野に入れて」）

  ROW0/1 は J_DB より上、ROW2/3/4 は下へ伸びる。行番号の昇順に並べると
  上下 2 群が必ず交差する（**実測 3 交差**）。群ごとに近い順で **0 交差**。
  そのズレは **XIAO のピン割り当て＝ファームで吸収**する（利用者の判断
  「配線でひねるのではなくソフトで受けるべき」）。

  ROW4 を D9 から左列へ戻した。右列へ逃がしていた理由は「左列が 6 本だと
  アンテナ直下を 2 本通る」だが、**その 6 本目は VBATT_SENSE だった。**
  分圧が子基板へ移って 5 本に戻ったので前提が消えた。
  → ファームの `&spi2_default`（MISO 外し）が**不要になり削除**。

■ アンテナの禁止域（利用者「こんなに広い必要ある？」「ズレてる」）

  子基板: 幅 18.3mm（XIAO の外形）を使っていた。**アンテナは 3.5mm 角**で
  4.1 倍。さらに y 方向に 2 つの細工（意味の無い切り詰めと水増し）があり、
  **アンテナの 57% しか覆っていなかった**。
    → `antenna_x_band()` に統一。**被覆 100%**、地板の無駄も消えた。
  主基板: アンテナから 3.9mm 外れた場所を抜いて 450mm² を捨てていた。
    → 削除（前のコミット）。

  ⚠️ **SES 往復でルール領域の層が消える**ことを発見した（GetLayer() が -1）。
  層を持たないゾーンは何も禁止しないので、あとから敷いたベタが
  アンテナ直下に入っていた（実測 3297 頂点）。`_restore_rule_area_layers`
  で戻す。**「宣言したから効いている」の 3 回目。**

■ 子基板を主基板と同じ水準に（利用者「MAIN にあって DB に無いもの」）

  両面 GND ベタ（裏面だけだった）・GND ファンアウト・スティッチング・
  離島の救済・電源のネットクラス。順序は **配置 → ネットクラス → 配線 →
  ベタ・ビア**（利用者「ベタは配線の残りで最大限やる」）。
  アンテナの禁止域だけは最初（配置と配線の制約なので）。

■ その他

  - バルクを縦置き＋向きを直した（V3V3/GND が XIAO と平行に並ぶ）
  - 行を D2〜D6 にして D1 を空け、奥側に 2.54mm 作った

■ 検査（どれも故意に壊して落ちることを確認）

  - `test_the_row_order_matches_between_firmware_and_circuit`
    行 N がファームと回路で同じピンを指すか。**既存の検査は集合しか
    見ておらず、D4 と D6 を入れ替えても通っていた**
  - 禁止域の寸法をアンテナの実寸と照合
  - `test_there_is_a_bulk_capacitor` を「XIAO と同じ基板にあるか」に
  - 変異検査が子基板も壊せるように（バルク移設で空振りしていた）
  - 正規表現がゾーンを跨いで**ベタ自身を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
Parts:
- added BT1_-: battery_land, symbol hhkb_split_daughterboard:battery_land
- added D_PWR: schottky, symbol hhkb_split_daughterboard:schottky
- added R_HI, R_LO: res_1M, symbol hhkb_split_daughterboard:res_1M
- added SW_PWR_1: wire_land, symbol hhkb_split_daughterboard:wire_land
Connections:
- net GND: now also BT1_-.1, R_LO.2
- net ROW0: now also J_MAIN.7, U_MCU.D2; no longer J_MAIN.8, U_MCU.D1
- net ROW1: now also J_MAIN.8, U_MCU.D3; no longer J_MAIN.9, U_MCU.D2
- net ROW2: now also J_MAIN.11, U_MCU.D6; no longer J_MAIN.10, U_MCU.D3
- net ROW3: now also J_MAIN.10, U_MCU.D5; no longer J_MAIN.11, U_MCU.D4
- net ROW4: now also J_MAIN.9, U_MCU.D4; no longer J_MAIN.4, U_MCU.D9
- net SPI_MOSI: now also J_MAIN.4; no longer J_MAIN.5
- net V3V3: now also J_MAIN.5, D_PWR.1 (K); no longer J_MAIN.6
- net VBATT_SENSE: now also D_PWR.2 (A), R_HI.1, R_HI.2, R_LO.1, SW_PWR_1.1; no longer J_MAIN.7
- no-connect marks 4 -> 5
Other:
- note added: "── 電源 ──"
- moved on the sheet: C_BULK, C_DB, J_MAIN, U_MCU
