File: pcb/matrix/hhkb_split_right.kicad_pcb (KiCad board)
At the start: 2 copper layers, 173.7 x 97.4 mm, 83 parts, among them SW1 CPG151101S11-2, SW10 CPG151101S11-2, SW11 CPG151101S11-2, SW12 CPG151101S11-2, SW13 CPG151101S11-2, SW14 CPG151101S11-2, SW15 CPG151101S11-2, SW16 CPG151101S11-2, SW17 CPG151101S11-2, SW18 CPG151101S11-2, SW19 CPG151101S11-2, SW2 CPG151101S11-2, SW20 CPG151101S11-2, SW21 CPG151101S11-2, SW22 CPG151101S11-2, SW23 CPG151101S11-2, SW24 CPG151101S11-2, SW25 CPG151101S11-2, SW26 CPG151101S11-2, SW27 CPG151101S11-2, SW28 CPG151101S11-2, SW29 CPG151101S11-2, SW3 CPG151101S11-2, SW30 CPG151101S11-2, SW31 CPG151101S11-2, SW32 CPG151101S11-2, SW33 CPG151101S11-2, SW34 CPG151101S11-2, SW4 CPG151101S11-2, SW5 CPG151101S11-2, SW6 CPG151101S11-2, SW7 CPG151101S11-2, SW8 CPG151101S11-2, SW9 CPG151101S11-2, U1 74LVC595, U2 74LVC595

Commit message: 左のキーマトリクスを完成させた（21 ホップ全部・DRC 0）
引けなかった 4 本を潰した。**どれも基板の都合ではなく、引き方が
硬かっただけ**だった（残っていた「障害物」は 4 本中 1 本も無い）。

足した形:
  C  跨いだあと、行の下で 45° に寄る
  C' 横が縦より長いとき、行の下を横に走ってから 45° で降りる
  D  跨いだ直後にレーンで横へ逃げてから降りる

踏んだ穴を注記に残した:
  - `knee < 0` を手前で弾いていて、そのために書いた C' が**一度も
    呼ばれていなかった**（左 COL3/COL5）
  - 行のバスは線ではなく**パッドの列**でもある。線だけ避けて K 側
    パッド（半対角 0.75mm）を 0.65mm で擦っていた（左 COL1/3/5）
  - 全列を同じ y のレーンに流して**自分どうしで交差**した
    （COL1/COL3/COL5 が y=124.000 に重なり tracks_crossing 2 件）。
    自分の障害物だけ見て、自分どうしを見ていなかった → 列ごとに
    レーンをずらす（LANE_PITCH）
  - C は縦の区間が元の x に長く残るので、スタビの穴（ST19 が列の
    x のほぼ真上）を抜けられなかった → D で先に横へ逃げる

左: 行 22 / 列 88 区間 / 橋のビア 42 個 / 引かなかったホップ 0。
配線由来の DRC 違反 0。残る未接続 17 件は全部 U1 / J_DB / C_U1 で、
キーとダイオードの間の未接続は 0（利用者の指示どおり MCU は無視）。

右は 6 ホップ残っている（別途）。

Co-Authored-By: Claude Opus 5 (1M context) <noreply@anthropic.com>
Routing:
- net COL7: track 23.0 -> 71.8 mm, vias 2 -> 4

Commit message: 最下段の列の配線を短くした（横断 164.44 → 89.79mm）
利用者の指摘「一番下の行だけ変ですね。そもそもそのキーがその列番号に
あることが妥当なのか、と言うところから疑って」。

**疑ったら、割り当ての方が間違っていた。**最下段は幅広キー
（Alt / Meta 1.5u / L-Space 3.0u）で、dtsi が **キーの真上を通らない列**
を選んでいる。実測: Meta は範囲 47.6〜76.2 に COL1/COL2 が通っている
のに COL3(90.5) を指定。L-Space は COL4 なら 4.76mm のところ COL5 で
14.29mm。**配線が長い横断になるのは当然だった。**

⚠️ **私は当初「割り当ては妥当」と報告したが誤りだった。**コードと
dtsi の一致しか見ておらず、**dtsi 自体（自分たちの生成物）が妥当かを
見ていなかった。**「自分の生成物どうしの一致は検証ではない」。

**ファームの修正は open-gaps #46 に記録した**（利用者「後でもできるので、
とりあえず配線を」）。ここでは配線側だけ短くする。

足した形と直した穴:
  E   下のキーの x で降ろし、横移動は行の上でやる（COL1 が採用）
  C'  **符号が逆で、目標を追い越してから戻っていた**（COL3 は
      x=117.1 まで行って 135.8 へ戻り、18.7mm 無駄にしていた）
  候補は**短い順に試す**。定義順だと先に書いた形が勝って長い経路が残る

左: 21 ホップ全部・列 88 区間・橋のビア 42 個・配線由来の DRC 違反 0。
未接続 17 件は全部 U1 / J_DB / C_U1（指示どおり MCU は無視）。
右は 4 ホップ残り（別途）。

Co-Authored-By: Claude Opus 5 (1M context) <noreply@anthropic.com>
Routing:
- net COL0: track 0.00 -> 28.6 mm, vias 0 -> 2
- net COL1: track 46.0 -> 72.9 mm, vias 4 -> 6
- net COL7: track 71.8 -> 56.3 mm

Commit message: 右の段 1 の列割り当てを規則的に直した（配線ルールは触らない）
利用者「右は、まず配線ルールは基本いじらずに、まずは列割り当てを
直しましょう。明らかに規則的じゃない」。

**測ったら、4 段のうち段 1 だけが不規則だった。**

段 1（Y U I O P [ ] Del）は列 8 を飛ばして 6,7,9,10,11,12,13,14 に
していた。**8 キーとも 1u で等間隔なのに途中で 1 つ飛ばすと、I 以降が
全部 1 列ぶん右にずれる**。実測で 2 キーが「キーの真上を通らない列」に
繋がっていた:

    P  範囲 257.2〜276.2  真上は COL10 だけ  なのに COL11(276.2)
    [  範囲 276.2〜295.3  真上は COL11 だけ  なのに COL12(295.3)

**6〜12 を連続で使い、空けるのは 13** に変更。これで 8 キーとも真上の
列に乗る（6/8 → 8/8）。Del だけ 1.5u で右端に寄るので COL14。

**他の段（2/3/4）は総当りで測った結果すでに最良**で、飛ばしている列は
幅広キー（Enter 2.25u / Shift 1.75u / R-Space 3u）による本物の欠番
だった。**触らない。**

配線ルールは 1 文字も変えていない。それでも割り当てを直しただけで
**引けなかったホップが 4 → 3 に減った**（右: 列 83 → 92 区間）。
配線由来の DRC 違反 0。残る未接続はマトリクス内 2 件（COL7/COL8）と
GND の島 1 件。

左は変化なし（段 1 は右だけの行。指紋で確認して戻した）。

Co-Authored-By: Claude Opus 5 (1M context) <noreply@anthropic.com>
Connections:
- SW12 pad 1: COL3 -> COL2
- SW13 pad 1: COL4 -> COL3
- SW14 pad 1: COL5 -> COL4
- SW15 pad 1: COL6 -> COL5
- SW16 pad 1: COL7 -> COL6
Routing:
- net COL2: track 44.0 -> 94.2 mm, vias 4 -> 8
- net COL7: track 56.3 -> 33.3 mm, vias 4 -> 2
- net COL6: track 44.0 -> 51.5 mm
- net COL5: track 65.0 -> 72.2 mm
- net COL4: track 86.1 -> 92.9 mm
- net COL3: track 67.0 -> 73.5 mm
- net COL0: track 28.6 -> 23.0 mm, vias 2 -> 0
- net COL1: vias 6 -> 4

Commit message: 右の列を「行内の順番＝列番号」にした（利用者の指定）
利用者「SW1, 10, 18, 25, 32 を Col 0 として。以降、その行を一つ右に
いくごとに列を増やして」「ただし SW33, 34 は例外」。

各行の左端が COL0、以降 +1。**飛ばさない。**以前は段ごとに開始列も
欠番もばらばらで（段2 は列 7 から、段4 は列 8 から、SW17 が COL8、
SW30 が COL7）、「行内の位置」と「列番号」が対応していなかった。

例外の SW33/SW34 は、実測でキーの真上を通る列に合わせた（確認済み）:
    SW33 Meta  範囲 247.65〜276.23 → COL3（x=261.94 と完全一致）
    SW34 Alt   範囲 276.23〜295.27 → COL4（ずれ 4.76mm）

**配線ルールは 1 文字も変えていない。**割り当てだけで、引けなかった
ホップが **4 → 2**、マトリクス内の未接続が **3 → 1** に減った
（右: 列 88 区間・橋のビア 38 個・配線由来の DRC 違反 0）。

## 検査を 1 つ作り直した

`test_matrix_columns_follow_physical_position`（同じ列のキーが x 方向に
1.5 キー幅以内）は、**この方針では必ず落ちる**——各行の左端が COL0 に
なるので同じ列が 38mm 散らばる。

**落ちるから外す、はしない。**守りたかったのは x の散らばりではなく
「長い横断が生まれないこと」（38mm の横断で DRC が交差を出した事故から
書かれた検査）なので、**そちらを直接測る**ように書き換えた
（`test_matrix_columns_do_not_need_long_crossings`）。実測の最長は
左 16.7mm / 右 20.2mm で、1 段ぶんの斜め（26.9mm）以内。

⚠️ **途中、正規表現が `(net <番号>)` を探していて 1 本も拾えず、
閾値を 15mm に下げても通っていた。**`(segment ...)` はネットを名前で
持つ。書式を実物で確かめて直し、**閾値を下げると落ちること**を
確認した（16.7 / 20.2mm が正しく出る）。読めなかったら落ちる
assert も足した。

本番の `pcb/` は古い割り当てのままなので
`test_matrix_wiring_matches_the_firmware` が赤。**意図した状態**として
open-gaps #47 に記録した（残り 6 件の赤は私の変更前から）。

Co-Authored-By: Claude Opus 5 (1M context) <noreply@anthropic.com>
Connections:
- SW17 pad 1: COL8 -> COL7
- SW18 pad 1: COL1 -> COL0
- SW19 pad 1: COL2 -> COL1
- SW20 pad 1: COL3 -> COL2
- SW21 pad 1: COL4 -> COL3
- SW22 pad 1: COL5 -> COL4
- SW23 pad 1: COL6 -> COL5
- SW24 pad 1: COL7 -> COL6
- SW25 pad 1: COL1 -> COL0
- SW26 pad 1: COL2 -> COL1
- SW27 pad 1: COL3 -> COL2
- SW28 pad 1: COL4 -> COL3
- SW29 pad 1: COL5 -> COL4
- SW30 pad 1: COL7 -> COL5
- SW31 pad 1: COL8 -> COL6
- SW32 pad 1: COL2 -> COL0
- SW33 pad 1: COL4 -> COL3
- SW34 pad 1: COL5 -> COL4
Routing:
- net COL0: track 23.0 -> 92.0 mm
- net COL2: track 94.2 -> 67.0 mm, vias 8 -> 6
- net COL8: track 21.0 -> 0.00 mm, vias 2 -> 0
- net COL5: track 72.2 -> 51.6 mm, vias 6 -> 4
- net COL3: track 73.5 -> 86.1 mm, vias 6 -> 8
- net COL1: track 72.9 -> 67.0 mm, vias 4 -> 6
- net COL4: track 92.9 -> 88.0 mm
- net COL6: track 51.5 -> 47.0 mm
- net COL7: track 33.3 -> 28.8 mm

Commit message: 右のマトリクスを完成させた（U1/U2 の移動を取り込み・引き残し 0）
利用者が基板上で U2 と U1 を動かした:
  「SW6 から SW15 は U2 をずらしたので、それで試してください」
  「SW16-24 は工夫して」
  「SW5, 6 だけど、他の同じ行の配線パターンを踏襲して」
  「コンデンサとか避けておいたので」

**U1/U2 の移動を生成器へ取り込んだ**（座標が完全一致することを確認）:
  U2  帯0 x=+15.0    → 帯1 x=-40.662 dy=+0.725  (109.338, 88.900)
  U1  帯0 x=+2.0     → 帯3 x=-75.938 dy=-0.025  ( 74.062,126.250)

どちらも**列の通り道を塞いでいた**。U2 は COL5（SW6→SW15）を、
U1 と C_U1 は COL4（x≈146〜152）を。移動で両方とも素直に降りられる。

**SW5 が同じ段の他と揃った**（利用者の指摘）。SW4/SW5/SW6 が
「0.200mm 降りて曲がり、75.650 で 45° を終える」と完全に同じ形。
前は SW5 だけ 3.700mm 降りていた（U1/C_U1 を避けるため）。

**SW16→SW24（ST24 のスタビ穴）は形 F で解いた。**C も D も曲がる y が
1 点に決まっており、そこが穴の真横だと 0.289mm しか空かない。
**曲がる高さを振れる形**を足すと、45° を保ったまま穴の左を抜けて
1.030mm 取れる（他の列と同じ値）。

2 つ直した:
  - 橋を架ける枝でも**余裕が最大の候補を採る**（他の枝は済んでいた）
  - `gen_matrix` が **GND の離島を繋いでいなかった**。配線が密になって
    ベタが割れ、DRC が「ゾーンが繋がっていない」を 2 件出した。
    本番と同じ `gnd_fanout.stitch_islands` を呼ぶ（左 10 個・右 12 個）。
    浮いた銅は 2.4GHz でアンテナになる

左右とも: **引かなかったホップ 0 / 配線由来の DRC 違反 0 /
マトリクス内の未接続 0 / 最小の隙間 1.030mm**。

⚠️ **C_U1 は取り込んでいない。**利用者の板では U1 から 136mm 離れており、
パスコンとして効かない位置（効くのは往復ループのインダクタンス）。
`DECOUPLE_BESIDE` が U1 から算出する仕組みのまま残した。

pytest の赤 8 件は**私の変更の前後で同じ**（本番 pcb/ が未再生成＝
open-gaps #47、SPARE 系は以前から）。

Co-Authored-By: Claude Opus 5 (1M context) <noreply@anthropic.com>
Parts:
- moved C_U1 96.6 mm to (68.2, 126.2)
- moved U1 96.6 mm to (74.1, 126.2)
- moved C_U2 59.1 mm to (103.4, 88.9)
- moved U2 59.1 mm to (109.3, 88.9)
Routing:
- net COL6: track 47.0 -> 79.8 mm, vias 4 -> 6
- net COL5: track 51.6 -> 73.3 mm, vias 4 -> 6
- net COL2: track 67.0 -> 70.7 mm
- net COL7: track 28.8 -> 26.7 mm
- net GND: vias 0 -> 12
